File: Kicad_Docs/OBDII_PIC_REVA/OBDII_PIC_REVA.kicad_sch (KiCad schematic)
At the start: 2 parts, among them U1 RC1602A-GHW-ESX, U2 PIC18F46K22-I_P

Commit message: kicad updated
Parts:
- added RV1: R_Potentiometer, symbol Device:R_Potentiometer
Connections:
- net GND: now reaches U1.1 (VSS)
- net GND: now also U1.10 (DB3), U1.16 (K), U1.4 (RS), U1.5 (R/~{W}), U1.7 (DB0), U1.8 (DB1), U1.9 (DB2), U1.K1 (K), RV1.1
- net RD4: now reaches U1.11 (DB4)
- net RD5: now reaches U1.12 (DB5)
- net RD6: now reaches U1.13 (DB6)
- net RD7: now reaches U1.14 (DB7)
- net +5V: now reaches U1.15 (A/VEE)
- net +5V: now also U1.2 (VDD), U1.A1 (A), RV1.3
- net Vo: now reaches U1.3 (Vo)
- net Vo: now also RV1.2
- net RD2: now reaches U1.6 (~{E})
- no-connect marks 0 -> 27
Other:
- moved on the sheet: U1

Commit message: kicad
Parts:
- added R1, R3: 10k, symbol Device:R
- added R2, R4: 1k, symbol Device:R
- added RV2: R_Potentiometer, symbol Device:R_Potentiometer
- added SW1, SW2: SW_MEC_5G, Button_Switch_SMD:SW_SPST_CK_KMS2xxGP, symbol Switch:SW_MEC_5G
Connections:
- net +5V: now also U2.11 (VDD), U2.32 (VDD), R1.1, R3.1, RV2.3
- net GND: now also U2.12 (VSS), U2.31 (VSS), RV2.1, SW1.1 (A), SW1.2 (A), SW2.1 (A), SW2.2 (A)
- net RD4: now also U2.27 (RD4/P2D/SDO2/AN24)
- net RD5: now also U2.28 (RD5/P1B/AN25)
- net RD6: now also U2.29 (RD6/P1C/TX2/CK2/AN26)
- net RD7: now also U2.30 (RD7/P1D/RX2/DT2/AN27)
- net RA0: now reaches U2.2 (RA0/C12IN0-/AN0)
- net RA0: now also RV2.2
- net RC5: now reaches U2.24 (RC5/SDO1/AN17)
- net RC5: now also R2.2
- net RC6_TXP_RXU: now reaches U2.25 (RC6/TX1/CK1/AN18)
- net RC7_RXP_TXU: now reaches U2.26 (RC7/RX1/DT1/AN19)
- net RB4: now reaches U2.37 (RB4/IOC0/T5G/AN11)
- net RB4: now also R4.2
- new net: R1.2, R2.1, SW1.3 (B), SW1.4 (B)
- new net: R3.2, R4.1, SW2.3 (B), SW2.4 (B)
Other:
- moved on the sheet: RV1, U1, U2

Commit message: Finished Schematic on KICAD
Parts:
- added U3: STN1110, symbol OBDII_UART:STN1110
Connections:
- net GND: now also U3.3 (GND)
- net RC6_TXP_RXU: now also U3.1 (UART_RX)
- net RC7_RXP_TXU: now also U3.1 (UART_RX)
Changed lines of the file:
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@@
+	)
+	(rectangle
+		(start 13.335 80.01)
+		(end 86.36 104.775)
+		(stroke
+			(width 0)
+			(type default)
+		)
+		(fill
+			(type none)
+		)
 	)
 	(rectangle
@@
 		(at 14.605 15.24 0)
 		(size 11.43 3.175)
+		(margins 0.9525 0.9525 0.9525 0.9525)
+		(stroke
+			(width 0)
+			(type solid)
+		)
+		(fill
+			(type none)
+		)
+		(effects
+			(font
+				(size 1.27 1.27)
+			)
+			(justify left top)
+		)
+	)
+	(text_box "When testing, you can use the Vbatt to 5v, however, before plugging the OBDII connector to the car, remove the Vbatt line so you dont kill the PIC"
+		(exclude_from_sim no)
+		(at 15.24 89.535 0)
+		(size 33.02 13.335)
+		(margins 0.9525 0.9525 0.9525 0.9525)
+		(stroke
+			(width 0)
+			(type solid)
+		)
+		(fill
+			(type none)
+		)
+		(effects
+			(font
+				(size 1.27 1.27)
+			)
+			(justify left top)
+		)
+	)
+	(text_box "Sparkfun_OBDII_to_UART"
+		(exclude_from_sim no)
+		(at 15.24 82.55 0)
+		(size 26.67 4.445)
 		(margins 0.9525 0.9525 0.9525 0.9525)
 		(stroke
@@
 	(wire
 		(pts
+			(xy 67.31 97.79) (xy 73.66 97.79)
+		)
+		(stroke
+			(width 0)
+			(type default)
+		)
+	)
+	(wire
+		(pts
 			(xy 40.64 45.72) (xy 45.72 45.72)
 		)
@@
 		)
 	)
+	(label "RC6_TXP_RXU"
+		(at 69.85 91.44 0)
+		(effects
+			(font
+				(size 1.27 1.27)
+			)
+			(justify left bottom)
+		)
+	)
 	(label "RD6"
 		(at 269.24 63.5 0)
@@
 	(label "RD2"
 		(at 92.71 31.75 0)
+		(effects
+			(font
+				(size 1.27 1.27)
+			)
+			(justify left bottom)
+		)
+	)
+	(label "RC7_RXP_TXU"
+		(at 69.85 88.9 0)
 		(effects
 			(font
@@
 	)
 	(symbol
+		(lib_id "power:GND")
+		(at 73.66 97.79 0)
+		(unit 1)
+		(exclude_from_sim no)
+		(in_bom yes)
+		(on_board yes)
+		(dnp no)
+		(fields_autoplaced yes)
+		(property "Reference" "#PWR016"
+			(at 73.66 104.14 0)
+			(effects
+				(font
+					(size 1.27 1.27)
+				)
+				(hide yes)
+			)
+		)
+		(property "Value" "GND"
+			(at 73.66 102.87 0)
+			(effects
+				(font
+					(size 1.27 1.27)
+				)
+			)
+		)
+		(property "Footprint" ""
+			(at 73.66 97.79 0)
+			(effects
+				(font
+					(size 1.27 1.27)
+				)
+				(hide yes)
+			)
+		)
+		(property "Datasheet" ""
+			(at 73.66 97.79 0)
+			(effects
+				(font
+					(size 1.27 1.27)
+				)
+				(hide yes)
+			)
+		)
+		(property "Description" "Power symbol creates a global label with name \"GND\" , ground"
+			(at 73.66 97.79 0)
+			(effects
+				(font
+					(size 1.27 1.27)
+				)
+				(hide yes)
+			)
+		)
+		(pin "1"
+		)
+		(instances
+			(project "OBDII_PIC_REVA"
+				(path "/82ea1033-e42f-45cf-b3f2-aacaaa1723fc"
+					(reference "#PWR016")
+					(unit 1)
+				)
+			)
+		)
+	)
+	(symbol
 		(lib_id "power:+5V")
 		(at 104.14 43.18 0)
@@
 					(unit 1)
 				)
+			)
+		)
+	)
+	(symbol
+		(lib_id "OBDII_UART:STN1110")
+		(at 60.96 92.71 0)
+		(unit 1)
+		(exclude_from_sim no)
+		(in_bom yes)
+		(on_board yes)
+		(dnp no)
+		(property "Reference" "U3"
+			(at 66.04 85.09 0)
+			(effects
+				(font
+					(size 1.27 1.27)
+				)
+			)
+		)
+		(property "Value" "STN1110"
+			(at 58.674 85.344 0)
+			(effects
+				(font
+					(size 1.27 1.27)
+				)
+			)
+		)
+		(property "Footprint" ""
+			(at 60.96 92.71 0)
+			(effects
+				(font
+					(size 1.27 1.27)
+				)
+				(hide yes)
+			)
+		)
+		(property "Datasheet" "https://www.scantool.net/scantool/downloads/234/stn1100-frpm-preliminary.pdf?srsltid=AfmBOoo-ck3aRutfNohtRgrJahpXeoSJl7bUUqXrZD0vmXV2ENzVUR-f"
+			(at 60.96 92.71 0)
+			(effects
+				(font
+					(size 1.27 1.27)
+				)
+				(hide yes)
+			)
+		)
+		(property "Description" ""
+			(at 60.96 92.71 0)
+			(effects
+				(font
+					(size 1.27 1.27)
+				)
+				(hide yes)
+			)
+		)
+		(pin "1"
+		)
+		(pin "1"
+		)
+		(pin "3"
+		)
+		(instances
+			(project ""
+				(path "/82ea1033-e42f-45cf-b3f2-aacaaa1723fc"
+					(reference "U3")
+					(unit 1)
+				)

Commit message: Updated Project Information
Added schematic to github
Added code to main page
Added explanation of modes and code setup
Added project requirements and features
Added Documentation links
Connections:
- net RC6_TXP_RXU: now also U3.2 (UART_RX); no longer U3.1 (UART_RX)
Changed lines of the file:
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@@
+	(wire
+		(pts
+			(xy 69.85 97.79) (xy 73.66 97.79)
+		)
+		(stroke
+			(width 0)
+			(type default)
+		)
+	)
 	(wire
 		(pts
@@
 		(pts
 			(xy 72.39 29.21) (xy 72.39 34.29)
-		)
-		(stroke
-			(width 0)
-			(type default)
-		)
-	)
-	(wire
-		(pts
-			(xy 67.31 97.79) (xy 73.66 97.79)
 		)
 		(stroke
@@
 			)
 		)
+		(pin "2"
+		)
 		(pin "1"
-		)
-		(pin "1"
